Commit message: further work on completing the stack. going to fake localisation for time sake.

File: openvslam/ros/src/bot_description/urdf/small_car.urdf (robot description, URDF)
Before this commit: robot small_car, 9 links, 8 joints
Links:
- removed link chassis
- added link base_link, mass 30.0; collision box size=.8 .4 .1; visual box size=.8 .4 .1
Joints:
- joint back_left_wheel_joint: parent chassis -> base_link
- joint back_right_wheel_joint: parent chassis -> base_link
- joint camera_joint_four: parent chassis -> base_link
- joint camera_joint_one: parent chassis -> base_link
- joint camera_joint_three: parent chassis -> base_link
- joint camera_joint_two: parent chassis -> base_link
- joint front_left_wheel_joint: parent chassis -> base_link
- joint front_right_wheel_joint: parent chassis -> base_link
